Commit message: fixed moments of inertia fixed xacro to load the inertia matrix correctly initial tests of the inverse pendulum in gazebo to free fall on push

File: inverse_pendulum_model/urdf/inverse_pendulum.xacro (robot description, xacro)
@@ -2,9 +2,11 @@
 <robot xmlns:xacro="http://www.ros.org/wiki/xacro"
        xmlns:controller="http://playerstage.sourceforge.net/gazebo/xmlschema/#controller"
+       xmlns:interface="http://playerstage.sourceforge.net/gazebo/xmlschema/#interface"
     name="inverse_pendulum">
     <!-- includes -->
     <xacro:include filename="$(find inverse_pendulum)/urdf/macros.xacro" />
+    <xacro:include filename="$(find inverse_pendulum)/urdf/properties.xacro" />
     <!-- colors -->
-    <gazebo reference="base">
+    <gazebo reference="foot">
         <material>Gazebo/Red</material>
     </gazebo>
@@ -25,38 +27,41 @@
         </plugin>
     </gazebo>
-    <!-- object properties -->
-    <!-- x-red, y-green, z-blue -->
-    <xacro:property name="foundation_width" value="0.5" />
-    <xacro:property name="foundation_depth" value="4.0" />
-    <xacro:property name="foundation_height" value="1.0" />
-    <xacro:property name="foundation_mass" value="" />
-    <link name="base">
+    <link name="root">
         <visual>
             <geometry>
                 <!-- x-red, y-green, z-blue -->
-                <box size="4 4 0.1" />
+                <box size="0.1 0.1 0.1" />
             </geometry>
-            <origin rpy="0 0 0" xyz="0 0 0.05" />
+            <origin rpy="0 0 0" xyz="0 0 0" />
+        </visual>
+    </link>
+    <joint name="root_to_foot" type="fixed">
+        <parent link="root" />
+        <child link="foot" />
+        <origin rpy="0 0 0" xyz="0 0 0" />
+    </joint>
+    <link name="foot">
+        <visual>
+            <geometry>
+                <!-- x-red, y-green, z-blue -->
+                <box size="${foot_width} ${foot_depth} ${foot_height}" />
+            </geometry>
+            <origin rpy="0 0 0" xyz="0 0 0" />
         </visual>
         <collision>
             <geometry>
-                <box size="4 4 0.1" />
+                <box size="${foot_width} ${foot_depth} ${foot_height}" />
             </geometry>
             <origin rpy="0 0 0" xyz="0 0 0" />
         </collision>
-        <inertial>
-            <pose>0 0 0 0 0 0</pose>
-            <inertia
-                ixx="0.01"
-                ixy="0.0"
-                ixz="0.0"
-                iyy="0.01"
-                iyz="0.0"
-                izz="0.1" />
-            <mass value="10.0" />
-        </inertial>
+        <xacro:inertial_matrix
+            mass="${foot_mass}"
+            x_length="${foot_width}"
+            y_length="${foot_depth}"
+            z_length="${foot_height}"
+        />
     </link>
-    <joint name="base_to_foundation" type="fixed">
-        <parent link="base" />
+    <joint name="foot_to_foundation" type="fixed">
+        <parent link="foot" />
         <child link="foundation" />
         <origin rpy="0 0 0" xyz="0 0 0.15" />
@@ -70,5 +75,5 @@
                            ${foundation_height}" />
             </geometry>
-            <origin rpy="0 0 0" xyz="0 0 0.6" />
+            <origin rpy="0 0 0" xyz="0 0 ${foot_height}" />
             <material name="blue">
                 <color rgba="0 0 1 1" />
@@ -81,7 +86,12 @@
                            ${foundation_height}" />
             </geometry>
-            <origin rpy="0 0 0" xyz="0 0 0.6" />
+            <origin rpy="0 0 0" xyz="0 0 ${foot_height}" />
         </collision>
-        <xacro:inertial_matrix mass="10" />
+        <xacro:inertial_matrix
+            mass="${foundation_mass}"
+            x_length="${foundation_width}"
+            y_length="${foundation_depth}"
+            z_length="${foundation_height}"
+            />
     </link>
     <joint name="foundation_to_connector" type="prismatic">
@@ -95,5 +105,7 @@
         <visual>
             <geometry>
-                <box size="0.2 0.2 0.2" />
+                <box size="${connector_width}
+                           ${connector_depth}
+                           ${connector_height}" />
             </geometry>
             <origin rpy="0 0 0" xyz="0 0 0" />
@@ -103,18 +115,20 @@
         </visual>
         <collision>
-            <!-- TODO: Tune this to more realistic values -->
             <geometry>
-                <box size="0.2 0.2 0.2" />
+                <box size="${connector_width}
+                           ${connector_depth}
+                           ${connector_height}" />
             </geometry>
             <origin rpy="0 0 0" xyz="0 0 0" />
         </collision>
-        <xacro:inertial_matrix mass="1" />
+        <xacro:inertial_matrix
+            mass="${connector_mass}"
+            x_length="${connector_width}"
+            y_length="${connector_depth}"
+            z_length="${connector_height}" />
     </link>
     <joint name="connector_to_arm" type="revolute">
         <parent link="connector" />
         <child link="arm" />
-        <!--
-        <origin rpy="-${90 * 3.14 / 180} 0 0" xyz="0 0 0.2"/>
-        -->
         <origin rpy="0 0 0" xyz="0 0 0.2" />
         <limit upper="${3.14/2}" lower="${-3.14/2}"
@@ -127,5 +141,7 @@
         <visual>
             <geometry>
-                <box size="0.2 0.2 2.5" />
+                <box size="${arm_width}
+                           ${arm_depth}
+                           ${arm_height}" />
             </geometry>
             <origin rpy="0 0 0" xyz="0 0 1.3" />
@@ -136,12 +152,20 @@
         <collision>
             <geometry>
-                <box size="0.2 0.2 2.5" />
+                <box size="${arm_width}
+                           ${arm_depth}
+                           ${arm_height}" />
             </geometry>
             <origin rpy="0 0 0" xyz="0 0 1.3" />
         </collision>
-        <xacro:inertial_matrix mass="200"/>
+        <xacro:inertial_matrix2
+            mass="${arm_mass}"
+            x_length="${arm_width}"
+            y_length="${arm_depth}"
+            z_length="${arm_height}" />
     </link>
     <!-- transmissions -->
     <xacro:transmission_block joint_name="foundation_to_connector" />
+    <!--
     <xacro:transmission_block joint_name="connector_to_arm" />
+    -->
 </robot>

File: inverse_pendulum_model/urdf/macros.xacro (robot description, xacro)
@@ -2,30 +2,5 @@
 <robot xmlns:xacro="http://www.ros.org/wiki/xacro"
     name="inverse_pendulum">
-    <!-- inertial tag for links -->
-    <!--
-         <xacro:macro name="inertial_matrix" params="mass width height depth">
-         -->
-    <xacro:macro name="inertial_matrix" params="mass">
-        <inertial>
-            <mass value="${mass}" />
-            <!-- https://en.wikipedia.org/wiki/List_of_moments_of_inertia -->
-            <inertia
-                ixx="0.01"
-                ixy="0.0"
-                ixz="0.0"
-                iyy="0.01"
-                iyz="0.0"
-                izz="0.01" />
-            <!--
-            <inertia
-                ixx="${1/12 * mass * ((heigth) ^ 2 + (depth ^ 2))}"
-                ixy="0.0"
-                ixz="0.0"
-                iyy="${1/12 * mass * ((width ^ 2) + (depth ^ 2))}"
-                iyz="0.0"
-                izz="${1/12 * mass * ((width ^ 2) + (height ^ 2))}" />
-                -->
-        </inertial>
-    </xacro:macro>
+    <!-- https://en.wikipedia.org/wiki/List_of_moments_of_inertia -->
     <xacro:macro name="transmission_block" params="joint_name">
         <transmission name="tran1">
@@ -44,3 +19,21 @@
         </transmission>
     </xacro:macro>
+    <xacro:macro name="inertial_matrix" params="mass x_length y_length z_length">
+      <inertial>
+        <mass value="${mass}" />
+        <origin xyz="0 0 0" />
+        <inertia ixx="${(1/12) * mass * (y_length*y_length + z_length*z_length)}" ixy="0.0" ixz="0.0"
+                 iyy="${(1/12) * mass * (x_length*x_length + z_length*z_length)}" iyz="0.0"
+                 izz="${(1/12) * mass * (x_length*x_length + y_length*y_length)}" />
+      </inertial>
+    </xacro:macro>
+    <xacro:macro name="inertial_matrix2" params="mass x_length y_length z_length">
+      <inertial>
+        <mass value="${mass}" />
+        <origin xyz="0 0 1.3" />
+        <inertia ixx="${(1/12) * mass * (y_length*y_length + z_length*z_length)}" ixy="0.0" ixz="0.0"
+                 iyy="${(1/12) * mass * (x_length*x_length + z_length*z_length)}" iyz="0.0"
+                 izz="${(1/12) * mass * (x_length*x_length + y_length*y_length)}" />
+      </inertial>
+    </xacro:macro>
 </robot>

Commit message: Added gazebo sensor imu to urdf

File: inverse_pendulum_model/urdf/inverse_pendulum.xacro (robot description, xacro)
@@ -164,6 +164,43 @@
             z_length="${arm_height}" />
     </link>
+    <joint name="arm_to_imu" type="fixed">
+        <parent link="arm" />
+        <child link="imu_link" />
+        <origin rpy="0 0 0" xyz="0 0 0" />
+        <axis xyz="0 0 0" rpy="0 0 0" />
+    </joint>
+    <link name="imu_link">
+        <visual>
+            <geometry>
+                <box size="0.2 0.2 0.2" />
+            </geometry>
+            <origin rpy="0 0 0" xyz="0 0 2.7" />
+            <material name="gray">
+                <color rgba="0.5 0.5 0.5 1" />
+            </material>
+        </visual>
+    </link>
     <!-- transmissions -->
     <xacro:transmission_block joint_name="foundation_to_connector" />
     <xacro:transmission_block joint_name="connector_to_arm" />
+    <gazebo reference="imu_link">
+        <gravity>true</gravity>
+        <sensor name="imu_sensor" type="imu">
+            <alwaysOn>true</alwaysOn>
+            <update_rate>100</update_rate>
+            <visualize>true</visualize>
+            <topic>__default_topic__</topic>
+            <plugin filename="libgazebo_ros_imu_sensor.so" name="imu_plugin">
+                <topicName>imu</topicName>
+                <bodyName>imu_link</bodyName>
+                <updateRateHZ>10.0</updateRateHZ>
+                <gaussianNoise>0.0</gaussianNoise>
+                <xyzOffset>0 0 0</xyzOffset>
+                <rpyOffset>0 0 0</rpyOffset>
+                <frameName>imu_link</frameName>
+                <initialOrientationAsReference>false</initialOrientationAsReference>
+            </plugin>
+            <pose>0 0 0 0 0 0</pose>
+        </sensor>
+    </gazebo>
 </robot>

Commit message: Added custom pluin for controlling the inverse pendulum

File: inverse_pendulum_model/urdf/inverse_pendulum.xacro (robot description, xacro)
@@ -167,5 +167,5 @@
         <parent link="arm" />
         <child link="imu_link" />
-        <origin rpy="0 0 0" xyz="0 0 0" />
+        <origin rpy="0 0 0" xyz="0 0 2.7" />
         <axis xyz="0 0 0" rpy="0 0 0" />
     </joint>
@@ -175,5 +175,5 @@
                 <box size="0.2 0.2 0.2" />
             </geometry>
-            <origin rpy="0 0 0" xyz="0 0 2.7" />
+            <origin rpy="0 0 0" xyz="0 0 0" />
             <material name="gray">
                 <color rgba="0.5 0.5 0.5 1" />
